Commit message: 。

File: rui/practice_ws/src/myrobot_description/urdf/turtlebot3_mecanum.urdf.xacro (robot description, xacro)
@@ -24,16 +24,18 @@
    		</visual>
 		<collision>
-			<origin xyz="0 0 0" rpy="0 0 0" />
-			<geometry>
-				<mesh filename="package://myrobot_description/meshes/bases/base_link.STL" />
-			</geometry>
-		</collision>
-		<inertial>
-			<origin xyz="0 0.055998 0.019157" rpy="0 0 0" />
-			<mass value="1.6718"/>
-	 		<inertia
-	 			ixx="0.01" ixy="0" ixz="0"
-				iyy="0.01" iyz="0"
-				izz="0.01" />
+			<!-- Use a convex chassis collision body for stable Gazebo contact. -->
+			<origin xyz="0.007 0 -0.002" rpy="0 0 0" />
+			<geometry>
+				<box size="0.185 0.145 0.045" />
+			</geometry>
+		</collision>
+		<inertial>
+			<!-- Keep the center of mass centered and below the wheel axles. -->
+			<origin xyz="0.007 0 -0.018" rpy="0 0 0" />
+			<mass value="2.20"/>
+	 		<inertia
+				ixx="0.0042" ixy="0" ixz="0"
+				iyy="0.0067" iyz="0"
+				izz="0.0100" />
 		</inertial>
 	</link>
@@ -57,14 +59,14 @@
 			<origin xyz="0 0 0" rpy="0 0 0" />
 			<geometry>
-				<mesh filename="package://myrobot_description/meshes/wheels/wheel_right_rear.STL" />
-			</geometry>
-		</collision>
-		<inertial>
-			<origin xyz="-0.1005 0.085 0" rpy="0 0 0" />
-			<mass value="0.31944"/>
-	 		<inertia
-	 			ixx="0.01" ixy="0" ixz="0"
-				iyy="0.01" iyz="0"
-				izz="0.01" />
+				<cylinder radius="0.033" length="0.018" />
+			</geometry>
+		</collision>
+		<inertial>
+			<origin xyz="0 0 0" rpy="0 0 0" />
+			<mass value="0.08"/>
+	 		<inertia
+				ixx="0.000022" ixy="0" ixz="0"
+				iyy="0.000022" iyz="0"
+				izz="0.000044" />
 		</inertial>
  	</link>
@@ -88,14 +90,14 @@
 			<origin xyz="0 0 0" rpy="0 0 0" />
 			<geometry>
-				<mesh filename="package://myrobot_description/meshes/wheels/wheel_left_rear.STL" />
-			</geometry>
-		</collision>
-		<inertial>
-			<origin xyz="-0.1005 0.085 0" rpy="0 0 0" />
-			<mass value="0.31944"/>
-	 		<inertia
-	 			ixx="0.01" ixy="0" ixz="0"
-				iyy="0.01" iyz="0"
-				izz="0.01" />
+				<cylinder radius="0.033" length="0.018" />
+			</geometry>
+		</collision>
+		<inertial>
+			<origin xyz="0 0 0" rpy="0 0 0" />
+			<mass value="0.08"/>
+	 		<inertia
+				ixx="0.000022" ixy="0" ixz="0"
+				iyy="0.000022" iyz="0"
+				izz="0.000044" />
 		</inertial>
  	</link>
@@ -119,14 +121,14 @@
 			<origin xyz="0 0 0" rpy="0 0 0" />
 			<geometry>
-				<mesh filename="package://myrobot_description/meshes/wheels/wheel_right_front.STL" />
-			</geometry>
-		</collision>
-		<inertial>
-			<origin xyz="0.1005 0 0" rpy="0 0 0" />
-			<mass value="0.31944"/>
-	 		<inertia
-	 			ixx="0.01" ixy="0" ixz="0"
-				iyy="0.01" iyz="0"
-				izz="0.01" />
+				<cylinder radius="0.033" length="0.018" />
+			</geometry>
+		</collision>
+		<inertial>
+			<origin xyz="0 0 0" rpy="0 0 0" />
+			<mass value="0.08"/>
+	 		<inertia
+				ixx="0.000022" ixy="0" ixz="0"
+				iyy="0.000022" iyz="0"
+				izz="0.000044" />
 		</inertial>
  	</link>
@@ -150,14 +152,14 @@
 			<origin xyz="0 0 0" rpy="0 0 0" />
 			<geometry>
-				<mesh filename="package://myrobot_description/meshes/wheels/wheel_left_front.STL" />
-			</geometry>
-		</collision>
-		<inertial>
-			<origin xyz="0.1005 0 0" rpy="0 0 0" />
-			<mass value="0.31944"/>
-	 		<inertia
-	 			ixx="0.01" ixy="0" ixz="0"
-				iyy="0.01" iyz="0"
-				izz="0.01" />
+				<cylinder radius="0.033" length="0.018" />
+			</geometry>
+		</collision>
+		<inertial>
+			<origin xyz="0 0 0" rpy="0 0 0" />
+			<mass value="0.08"/>
+	 		<inertia
+				ixx="0.000022" ixy="0" ixz="0"
+				iyy="0.000022" iyz="0"
+				izz="0.000044" />
 		</inertial>
  	</link>
@@ -205,6 +207,6 @@
   <gazebo reference="wheel_right_rear">
     <material>Gazebo/Black</material>
-    <mu1>1.0</mu1>
-    <mu2>1.0</mu2>
+    <mu1>0.55</mu1>
+    <mu2>0.55</mu2>
     <kp>100000.0</kp>
     <kd>1.0</kd>
@@ -212,6 +214,6 @@
   <gazebo reference="wheel_left_rear">
     <material>Gazebo/Black</material>
-    <mu1>1.0</mu1>
-    <mu2>1.0</mu2>
+    <mu1>0.55</mu1>
+    <mu2>0.55</mu2>
     <kp>100000.0</kp>
     <kd>1.0</kd>
@@ -219,6 +221,6 @@
   <gazebo reference="wheel_right_front">
     <material>Gazebo/Blue</material>
-    <mu1>1.0</mu1>
-    <mu2>1.0</mu2>
+    <mu1>0.55</mu1>
+    <mu2>0.55</mu2>
     <kp>100000.0</kp>
     <kd>1.0</kd>
@@ -226,6 +228,6 @@
   <gazebo reference="wheel_left_front">
     <material>Gazebo/Blue</material>
-    <mu1>1.0</mu1>
-    <mu2>1.0</mu2>
+    <mu1>0.55</mu1>
+    <mu2>0.55</mu2>
     <kp>100000.0</kp>
     <kd>1.0</kd>
